Commit message: init

File: racebot_description/urdf/mecanum/mecanum_base.xacro (robot description, xacro)
@@ -1,58 +1,60 @@
-<?xml version="1.0" ?>
+<?xml version="1.0"?>
 <robot name="mecanum_base" xmlns:xacro="http://www.ros.org/wiki/xacro">
     <material name="blue">
-        <color rgba="0 0 0.8 1"/>
+        <color rgba="0 0 0.8 1" />
     </material>
     <material name="black">
-        <color rgba="0 0 0 1"/>
+        <color rgba="0 0 0 1" />
     </material>
     <material name="white">
-        <color rgba="1 1 1 1"/>
+        <color rgba="1 1 1 1" />
     </material>
     <material name="red">
-        <color rgba="0.8 0.0 0.0 1.0"/>
+        <color rgba="0.8 0.0 0.0 1.0" />
+    </material>
+    <material name="grey">
+        <color rgba="0 0 0 0.5" />
     </material>
     <xacro:macro name="default_inertial" params="mass">
         <inertial>
-            <mass value="${mass}"/>
-            <inertia ixx="1.0" ixy="0.0" ixz="0.0" iyy="1.0" iyz="0.0" izz="1.0"/>
+            <mass value="${mass}" />
+            <inertia ixx="1.0" ixy="0.0" ixz="0.0" iyy="1.0" iyz="0.0" izz="1.0" />
         </inertial>
     </xacro:macro>
     <xacro:macro name="mecanum_base">
-        <link name="base_footprint"/>
+        <link name="base_footprint" />
         <link name="base_link">
             <inertial>
-                <mass value="10.69655"/>
-                <origin rpy="0 0 0 " xyz="0 0 0"/>
-                <inertia ixx="1.387114121" ixy="0" ixz="0" iyy="1.566123162" iyz="0" izz="0.343148801"/>
-            </inertial>
-            <collision>
-                <origin rpy="0 0 0" xyz="0 0 0"/>
-                <geometry>
-                    <box size="0.28 0.1 0.03"/>
-                </geometry>
-            </collision>
-            <visual>
-                <origin rpy="0 0 0" xyz="0 0 0"/>
-                <geometry>
-                    <box size="0.28 0.1 0.03"/>
-                </geometry>
-                <material name="base_link">
-                    <color rgba="0.0 0.0 0.8 1" />
-                </material>
+                <mass value="10.69655" />
+                <origin rpy="0 0 0 " xyz="0 0 0" />
+                <inertia ixx="1.387114121" ixy="0" ixz="0" iyy="1.566123162" iyz="0"
+                    izz="0.343148801" />
+            </inertial>
+            <collision>
+                <origin rpy="0 0 0" xyz="0 0 0" />
+                <geometry>
+                    <box size="0.9 0.6 0.1" />
+                </geometry>
+            </collision>
+            <visual>
+                <origin rpy="0 0 0" xyz="0 0 0" />
+                <geometry>
+                    <box size="0.9 0.6 0.1" />
+                </geometry>
+                <material name="black" />
             </visual>
         </link>
         <joint name="base_joint" type="fixed">
-            <origin xyz="0 0 -0.0288" rpy="0 0 0" />
-            <parent link="base_link"/>
+            <origin xyz="0 0 -0.05" rpy="0 0 0" />
+            <parent link="base_link" />
             <child link="base_footprint" />
         </joint>
         <joint name="join_left_front" type="fixed">
             <!-- <origin xyz="0.1825 0.195 0.049" rpy="0 0 1.57"/> -->
-            <parent link="base_link"/>
-            <child link="link_left_front"/>
+            <parent link="base_link" />
+            <child link="link_left_front" />
             <!-- <axis xyz="1 0 0" />
             <limit effort="30" velocity="17.4" /> -->
-            <origin xyz="0.13 0.09 0" />
+            <origin xyz="0.40 0.33 0" />
             <axis xyz="0 1 0" />
             <limit effort="10" velocity="1000" />
@@ -61,32 +63,32 @@
             <pose>0 0 0 0 0 0</pose>
             <inertial>
-                <mass value="0.59"/>
-                <!--<origin xyz="0 0 0" rpy="0 0 0"/>-->
-                <origin xyz="0 0 -0.07625" rpy="0 0 -1.57"/>
-                <inertia ixx="0.002525266" ixy="0" ixz="0" iyy="0.001311197" iyz="0" izz="0.001311136"/>
-            </inertial>
-            <collision>
-                <origin xyz="0 0 0" rpy="1.57 0 0" />
-                <geometry>
-                    <cylinder radius="0.033" length="0.02" />
-                </geometry>
-            </collision>
-            <visual>
-                <origin xyz="0 0 0" rpy="1.57 0 0" />
-                <geometry>
-                    <cylinder radius="0.033" length="0.02" />
-                </geometry>
-                <material name="wheels">
-                    <color rgba="0.6 0.6 0.6 1" />
-                </material>
+                <mass value="0.59" />
+                <!--<origin
+                xyz="0 0 0" rpy="0 0 0"/>-->
+                <origin xyz="0 0 -0.07625" rpy="0 0 -1.57" />
+                <inertia ixx="0.002525266" ixy="0" ixz="0" iyy="0.001311197" iyz="0"
+                    izz="0.001311136" />
+            </inertial>
+            <collision>
+                <origin xyz="0 0 0" rpy="1.57 0 0" />
+                <geometry>
+                    <cylinder radius="0.05" length="0.03" />
+                </geometry>
+            </collision>
+            <visual>
+                <origin xyz="0 0 0" rpy="1.57 0 0" />
+                <geometry>
+                    <cylinder radius="0.05" length="0.03" />
+                </geometry>
+                <material name="white" />
             </visual>
         </link>
         <joint name="join_right_front" type="fixed">
             <!-- <origin xyz="0.1825 -0.195 0.049" rpy="0 0 1.57"/> -->
-            <parent link="base_link"/>
-            <child link="link_right_front"/>
+            <parent link="base_link" />
+            <child link="link_right_front" />
             <!-- <axis xyz="1 0 0" /> -->
             <!-- <limit effort="30" velocity="17.4" /> -->
-            <origin xyz="0.13 -0.09 0" />
+            <origin xyz="0.40 -0.33 0" />
             <axis xyz="0 1 0" />
             <limit effort="10" velocity="1000" />
@@ -95,32 +97,32 @@
             <pose>0 0 0 0 0 0</pose>
             <inertial>
-                <mass value="0.59"/>
-                <!--<origin xyz="0 0 0" rpy="0 0 0"/>-->
-                <origin xyz="0 0 -0.07625" rpy="0 0 -1.57"/>
-                <inertia ixx="0.002525266" ixy="0" ixz="0" iyy="0.001311197" iyz="0" izz="0.001311136"/>
-            </inertial>
-            <collision>
-                <origin xyz="0 0 0" rpy="1.57 0 0" />
-                <geometry>
-                    <cylinder radius="0.033" length="0.02" />
-                </geometry>
-            </collision>
-            <visual>
-                <origin xyz="0 0 0" rpy="1.57 0 0" />
-                <geometry>
-                    <cylinder radius="0.033" length="0.02" />
-                </geometry>
-                <material name="wheels">
-                    <color rgba="0.6 0.6 0.6 1" />
-                </material>
+                <mass value="0.59" />
+                <!--<origin
+                xyz="0 0 0" rpy="0 0 0"/>-->
+                <origin xyz="0 0 -0.07625" rpy="0 0 -1.57" />
+                <inertia ixx="0.002525266" ixy="0" ixz="0" iyy="0.001311197" iyz="0"
+                    izz="0.001311136" />
+            </inertial>
+            <collision>
+                <origin xyz="0 0 0" rpy="1.57 0 0" />
+                <geometry>
+                    <cylinder radius="0.05" length="0.03" />
+                </geometry>
+            </collision>
+            <visual>
+                <origin xyz="0 0 0" rpy="1.57 0 0" />
+                <geometry>
+                    <cylinder radius="0.05" length="0.03" />
+                </geometry>
+                <material name="white" />
             </visual>
         </link>
         <joint name="join_left_back" type="fixed">
             <!-- <origin xyz="-0.1825 0.195 0.049" rpy="0 0 1.57"/> -->
-            <parent link="base_link"/>
-            <child link="link_left_back"/>
+            <parent link="base_link" />
+            <child link="link_left_back" />
             <!-- <axis xyz="1 0 0" /> -->
             <!-- <limit effort="30" velocity="17.4" /> -->
-            <origin xyz="-0.13 0.09 0" />
+            <origin xyz="-0.40 0.33 0" />
             <axis xyz="0 1 0" />
             <limit effort="10" velocity="1000" />
@@ -129,32 +131,32 @@
             <pose>0 0 0 0 0 0</pose>
             <inertial>
-                <mass value="0.59"/>
-                <!--<origin xyz="0 0 0" rpy="0 0 0"/>-->
-                <origin xyz="0 0 -0.07625" rpy="0 0 -1.57"/>
-                <inertia ixx="0.002525266" ixy="0" ixz="0" iyy="0.001311197" iyz="0" izz="0.001311136"/>
-            </inertial>
-            <collision>
-                <origin xyz="0 0 0" rpy="1.57 0 0" />
-                <geometry>
-                    <cylinder radius="0.033" length="0.02" />
-                </geometry>
-            </collision>
-            <visual>
-                <origin xyz="0 0 0" rpy="1.57 0 0" />
-                <geometry>
-                    <cylinder radius="0.033" length="0.02" />
-                </geometry>
-                <material name="wheels">
-                    <color rgba="0.6 0.6 0.6 1" />
-                </material>
+                <mass value="0.59" />
+                <!--<origin
+                xyz="0 0 0" rpy="0 0 0"/>-->
+                <origin xyz="0 0 -0.07625" rpy="0 0 -1.57" />
+                <inertia ixx="0.002525266" ixy="0" ixz="0" iyy="0.001311197" iyz="0"
+                    izz="0.001311136" />
+            </inertial>
+            <collision>
+                <origin xyz="0 0 0" rpy="1.57 0 0" />
+                <geometry>
+                    <cylinder radius="0.05" length="0.03" />
+                </geometry>
+            </collision>
+            <visual>
+                <origin xyz="0 0 0" rpy="1.57 0 0" />
+                <geometry>
+                    <cylinder radius="0.05" length="0.03" />
+                </geometry>
+                <material name="white" />
             </visual>
         </link>
         <joint name="join_right_back" type="fixed">
             <!-- <origin xyz="-0.1825 -0.195 0.049" rpy="0 0 1.57"/> -->
-            <parent link="base_link"/>
-            <child link="link_right_back"/>
+            <parent link="base_link" />
+            <child link="link_right_back" />
             <!-- <axis xyz="1 0 0" /> -->
             <!-- <limit effort="30" velocity="17.4" /> -->
-            <origin xyz="-0.13 -0.09 0" />
+            <origin xyz="-0.40 -0.33 0" />
             <axis xyz="0 1 0" />
             <limit effort="10" velocity="1000" />
@@ -163,143 +165,160 @@
             <pose>0 0 0 0 0 0</pose>
             <inertial>
-                <mass value="0.59"/>
-                <!--<origin xyz="0 0 0" rpy="0 0 0"/>-->
-                <origin xyz="0 0 -0.07625" rpy="0 0 -1.57"/>
-                <inertia ixx="0.002525266" ixy="0" ixz="0" iyy="0.001311197" iyz="0" izz="0.001311136"/>
-            </inertial>
-            <collision>
-                <origin xyz="0 0 0" rpy="1.57 0 0" />
-                <geometry>
-                    <cylinder radius="0.033" length="0.02" />
-                </geometry>
-            </collision>
-            <visual>
-                <origin xyz="0 0 0" rpy="1.57 0 0" />
-                <geometry>
-                    <cylinder radius="0.033" length="0.02" />
-                </geometry>
-                <material name="wheels">
-                    <color rgba="0.6 0.6 0.6 1" />
-                </material>
-            </visual>
-        </link>
-    <link name="lidar">
-        <visual>
-            <geometry>
-                <cylinder radius="0.03" length="0.06" />
-            </geometry>
-            <origin xyz="0 0 0" rpy="0 0 0" />
-            <material name="black">
-                <color rgba="0.0 0.0 0.0 1.0" />
-            </material>
-        </visual>
-        <collision>
-            <geometry>
-                <cylinder radius="0.03" length="0.06" />
-            </geometry>
-            <origin xyz="0.0 0.0 0.0" rpy="0.0 0.0 0.0" />
-        </collision>
-        <inertial>
-            <origin xyz="0 0 0" />
-            <mass value="0.1" />
-            <inertia ixx="6.64E-04" ixy="0" ixz="0" iyy="6.64E-04" iyz="0" izz="1.02E-03" />
-        </inertial>
-    </link>
-    <joint name="lidar_joint" type="fixed">
-        <parent link="base_link" />
-        <child link="lidar" />
-        <origin xyz="0.093603 0 0.12377" />
-        <axis xyz="0 0 1" />
-    </joint>
-    <link name="camera">
-        <visual>
-            <geometry>
-                <box size="0.005 0.03 0.03"/>
-            </geometry>
-            <origin xyz="0 0 0" rpy="0 0 0" />
-            <material name="black">
-                <color rgba="0.0 0.0 0.0 1.0" />
-            </material>
-        </visual>
-        <collision>
-            <geometry>
-                <box size="0.005 0.03 0.03"/>
-            </geometry>
-            <origin xyz="0.0 0.0 0.0" rpy="0.0 0.0 0.0" />
-        </collision>
-        <inertial>
-            <origin xyz="0 0 0" />
-            <mass value="0.05" />
-            <inertia ixx="6.64E-04" ixy="0" ixz="0" iyy="6.64E-04" iyz="0" izz="1.02E-03" />
-        </inertial>
-    </link>
-    <joint name="camera_joint" type="fixed">
-        <parent link="base_link" />
-        <child link="camera" />
-        <origin xyz="0.14851 0.0022137 0.0975" />
-        <axis xyz="0 0 1" />
-    </joint>
-    <link name="real_sense">
-        <visual>
-            <geometry>
-                <box size="0.01 0.1 0.02"/>
-            </geometry>
-            <origin xyz="0 0 0" rpy="0 0 0" />
-            <material name="black">
-                <color rgba="0.0 0.0 0.0 1.0" />
-            </material>
-        </visual>
-        <collision>
-            <geometry>
-                <box size="0.01 0.1 0.02"/>
-            </geometry>
-            <origin xyz="0.0 0.0 0.0" rpy="0.0 0.0 0.0" />
-        </collision>
-        <inertial>
-            <origin xyz="0 0 0" />
-            <mass value="0.05" />
-            <inertia ixx="6.64E-04" ixy="0" ixz="0" iyy="6.64E-04" iyz="0" izz="1.02E-03" />
-        </inertial>
-    </link>
-    <joint name="realsense_joint" type="fixed">
-        <parent link="base_link" />
-        <child link="real_sense" />
-        <origin xyz="0.19864 0.0038046 0.052021" />
-        <axis xyz="0 0 1" />
-    </joint>
-    <link name="realsense_depth"/>
-    <joint name="realsense_depth_joint" type="fixed">
-            <origin xyz="0 0 0" rpy="-1.5708 0 -1.5708"/>
-            <parent link="real_sense"/>
-            <child link="realsense_depth"/>
-    </joint>
-    <link name="imu">
-        <visual>
-            <geometry>
-                <box size="0.01 0.01 0.005"/>
-            </geometry>
-            <origin xyz="0 0 0" rpy="0 0 0" />
-            <material name="black">
-                <color rgba="0.0 0.0 0.0 1.0" />
-            </material>
-        </visual>
-        <collision>
-            <geometry>
-                <box size="0.01 0.01 0.005"/>
-            </geometry>
-            <origin xyz="0.0 0.0 0.0" rpy="0.0 0.0 0.0" />
-        </collision>
-        <inertial>
-            <origin xyz="0 0 0" />
-            <mass value="0.05" />
-            <inertia ixx="6.64E-04" ixy="0" ixz="0" iyy="6.64E-04" iyz="0" izz="1.02E-03" />
-        </inertial>
-    </link>
-    <joint name="imu_joint" type="fixed">
-        <parent link="base_link" />
-        <child link="imu" />
-        <origin xyz="0 0 0.02" />
-        <axis xyz="0 0 1" />
-    </joint>
+                <mass value="0.59" />
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