Commit message: add mecanum

File: racebot_description/urdf/ackermann/ackermanncar.xacro (robot description, xacro)
@@ -8,5 +8,4 @@
             <geometry>
                 <box size="0.28 0.1 0.03"/>
-                <!-- <mesh filename="package://tianracer_description/meshes/base_link.STL" /> -->
             </geometry>
             <!-- <origin xyz="0 0 -0.023" rpy="0 0 0" /> -->
@@ -102,5 +101,5 @@
     </joint>
      <xacro:wheel_transmission name="left_front_wheel" />
-<link name="right_steering_hinge">
+    <link name="right_steering_hinge">
         <visual>
             <geometry>
@@ -132,5 +131,5 @@
     </joint>
     <xacro:steering_hinge_transmission name="right_steering_hinge" />
-     <link name="right_front_wheel">
+    <link name="right_front_wheel">
         <visual>
             <geometry>
@@ -340,4 +339,4 @@
         <axis xyz="0 0 1" />
     </joint>
-  <xacro:include filename="$(find racebot_description)/urdf/ackermann/racecar.gazebo" />
+  <xacro:include filename="$(find racebot_description)/urdf/ackermann/ackermanncar.gazebo" />
 </robot>

Commit message: init

File: racebot_description/urdf/ackermann/ackermanncar.xacro (robot description, xacro)
@@ -11,6 +11,6 @@
             <!-- <origin xyz="0 0 -0.023" rpy="0 0 0" /> -->
             <origin xyz="0 0 0" rpy="0 0 0" />
-            <material name="yellow">
-                <color rgba="0.8 0.3 0.1 0.5" />
+            <material name="white">
+                <color rgba="1 1 1 1" />
             </material>
         </visual>

Commit message: ackermann

File: racebot_description/urdf/ackermann/ackermanncar.xacro (robot description, xacro)
@@ -2,4 +2,19 @@
 <robot name="racebot" xmlns:xacro="http://www.ros.org/wiki/xacro">
     <xacro:include filename="$(find racebot_description)/urdf/ackermann/macros.xacro" />
+    <material name="blue">
+        <color rgba="0 0 0.8 1" />
+    </material>
+    <material name="black">
+        <color rgba="0 0 0 1" />
+    </material>
+    <material name="white">
+        <color rgba="1 1 1 1" />
+    </material>
+    <material name="red">
+        <color rgba="0.8 0.0 0.0 1.0" />
+    </material>
+    <material name="grey">
+        <color rgba="0 0 0 0.5" />
+    </material>
     <link name="base_footprint">
     </link>
@@ -7,15 +22,12 @@
         <visual>
             <geometry>
-                <box size="0.28 0.1 0.03"/>
-            </geometry>
-            <!-- <origin xyz="0 0 -0.023" rpy="0 0 0" /> -->
-            <origin xyz="0 0 0" rpy="0 0 0" />
-            <material name="yellow">
-                <color rgba="0.8 0.3 0.1 0.5" />
-            </material>
-        </visual>
-        <collision>
-            <geometry>
-                <box size="0.28 0.1 0.03" />
+                <box size="0.9 0.6 0.1" />
+            </geometry>
+            <origin xyz="0 0 0" rpy="0 0 0" />
+            <material name="black" />
+        </visual>
+        <collision>
+            <geometry>
+                <box size="0.9 0.6 0.1" />
             </geometry>
             <origin xyz="0.0 0.0 0.0" rpy="0.0 0.0 0.0" />
@@ -24,9 +36,9 @@
     <joint name="base_link2base_footprint" type="fixed">
         <parent link="base_footprint" />
-        <child link="base_link"/>
-        <origin xyz="0 0 0.032" rpy="0 0 0" />
+        <child link="base_link" />
+        <origin xyz="0 0 -0.05" rpy="0 0 0" />
     </joint>
     <link name="base_inertia">
-    <inertial>
+        <inertial>
             <origin xyz="0 0 0" />
             <mass value="4" />
@@ -35,8 +47,8 @@
     </link>
     <joint name="chassis_inertia_joint" type="fixed">
-    <origin xyz="0 0 0" rpy="0 0 0" />
-    <parent link="base_link" />
-    <child link="base_inertia" />
-  </joint>
+        <origin xyz="0 0 0" rpy="0 0 0" />
+        <parent link="base_link" />
+        <child link="base_inertia" />
+    </joint>
     <link name="left_steering_hinge">
         <visual>
@@ -66,7 +78,7 @@
         <parent link="base_link" />
         <child link="left_steering_hinge" />
-        <origin xyz="0.13 0.065 0" />
-        <axis xyz="0 0 1" />
-        <limit lower="-0.6" upper="0.6" effort="5.0" velocity="1000.0"/>
+        <origin xyz="0.40 0.33 0" />
+        <axis xyz="0 0 1" />
+        <limit lower="-0.8" upper="0.8" effort="5.0" velocity="1000.0" />
     </joint>
     <xacro:steering_hinge_transmission name="left_steering_hinge" />
@@ -74,14 +86,12 @@
         <visual>
             <geometry>
-                <cylinder radius="0.033" length="0.02" />
-            </geometry>
-            <origin xyz="0 0 0" rpy="1.57 0 0" />
-            <material name="black">
-                <color rgba="0.0 0.0 0.0 1.0" />
-            </material>
-        </visual>
-        <collision>
-            <geometry>
-                <cylinder radius="0.032" length="0.02" />
+                <cylinder radius="0.075" length="0.03" />
+            </geometry>
+            <origin xyz="0 0 0" rpy="1.57 0 0" />
+            <material name="white" />
+        </visual>
+        <collision>
+            <geometry>
+                <cylinder radius="0.075" length="0.03" />
             </geometry>
             <origin xyz="0.0 0.0 0.0" rpy="1.57 0.0 0.0" />
@@ -100,14 +110,12 @@
         <limit effort="10" velocity="1000" />
     </joint>
-     <xacro:wheel_transmission name="left_front_wheel" />
+    <xacro:wheel_transmission name="left_front_wheel" />
     <link name="right_steering_hinge">
         <visual>
             <geometry>
-                 <cylinder radius="0.01" length="0.005" />
-            </geometry>
-            <origin xyz="0 0 0" rpy="1.57 0 0" />
-            <material name="black">
-                <color rgba="0.0 0.0 0.0 1.0" />
-            </material>
+                <cylinder radius="0.01" length="0.005" />
+            </geometry>
+            <origin xyz="0 0 0" rpy="1.57 0 0" />
+            <material name="black" />
         </visual>
         <collision>
@@ -126,7 +134,7 @@
         <parent link="base_link" />
         <child link="right_steering_hinge" />
-        <origin xyz="0.13 -0.065 0" />
-        <axis xyz="0 0 1" />
-        <limit lower="-0.6" upper="0.6" effort="5.0" velocity="1000.0"/>
+        <origin xyz="0.40 -0.33 0" />
+        <axis xyz="0 0 1" />
+        <limit lower="-0.8" upper="0.8" effort="5.0" velocity="1000.0" />
     </joint>
     <xacro:steering_hinge_transmission name="right_steering_hinge" />
@@ -134,14 +142,12 @@
         <visual>
             <geometry>
-                <cylinder radius="0.033" length="0.02" />
-            </geometry>
-            <origin xyz="0 0 0" rpy="1.57 0 0" />
-            <material name="black">
-                <color rgba="0.0 0.0 0.0 1.0" />
-            </material>
-        </visual>
-        <collision>
-            <geometry>
-                <cylinder radius="0.032" length="0.02" />
+                <cylinder radius="0.075" length="0.03" />
+            </geometry>
+            <origin xyz="0 0 0" rpy="1.57 0 0" />
+            <material name="white" />
+        </visual>
+        <collision>
+            <geometry>
+                <cylinder radius="0.075" length="0.03" />
             </geometry>
             <origin xyz="0.0 0.0 0.0" rpy="1.57 0.0 0.0" />
@@ -164,14 +170,12 @@
         <visual>
             <geometry>
-                <cylinder radius="0.032" length="0.02" />
-            </geometry>
-            <origin xyz="0 0 0" rpy="1.57 0 0" />
-            <material name="black">
-                <color rgba="0.0 0.0 0.0 1.0" />
-            </material>
-        </visual>
-        <collision>
-            <geometry>
-                <cylinder radius="0.032" length="0.02" />
+                <cylinder radius="0.075" length="0.03" />
+            </geometry>
+            <origin xyz="0 0 0" rpy="1.57 0 0" />
+            <material name="white" />
+        </visual>
+        <collision>
+            <geometry>
+                <cylinder radius="0.075" length="0.03" />
             </geometry>
             <origin xyz="0.0 0.0 0.0" rpy="1.57 0.0 0.0" />
@@ -186,5 +190,5 @@
         <parent link="base_link" />
         <child link="left_rear_wheel" />
-        <origin xyz="-0.13 0.09 0" />
+        <origin xyz="-0.40 0.33 0" />
         <axis xyz="0 1 0" />
         <limit effort="10" velocity="1000" />
@@ -194,14 +198,12 @@
         <visual>
             <geometry>
-                <cylinder radius="0.032" length="0.02" />
-            </geometry>
-            <origin xyz="0 0 0" rpy="1.57 0 0" />
-            <material name="black">
-                <color rgba="0.0 0.0 0.0 1.0" />
-            </material>
-        </visual>
-        <collision>
-            <geometry>
-                <cylinder radius="0.032" length="0.02" />
+                <cylinder radius="0.075" length="0.03" />
+            </geometry>
+            <origin xyz="0 0 0" rpy="1.57 0 0" />
+            <material name="white" />
+        </visual>
+        <collision>
+            <geometry>
+                <cylinder radius="0.075" length="0.03" />
             </geometry>
             <origin xyz="0.0 0.0 0.0" rpy="1.57 0.0 0.0" />
@@ -216,5 +218,5 @@
         <parent link="base_link" />
         <child link="right_rear_wheel" />
-        <origin xyz="-0.13 -0.09 0" />
+        <origin xyz="-0.40 -0.33 0" />
         <axis xyz="0 1 0" />
         <limit effort="10" velocity="1000" />
@@ -224,14 +226,12 @@
         <visual>
             <geometry>
-                <box size="0.005 0.03 0.03"/>
-            </geometry>
-            <origin xyz="0 0 0" rpy="0 0 0" />
-            <material name="black">
-                <color rgba="0.0 0.0 0.0 1.0" />
-            </material>
-        </visual>
-        <collision>
-            <geometry>
-                <box size="0.005 0.03 0.03"/>
+                <box size="0.005 0.03 0.03" />
+            </geometry>
+            <origin xyz="0 0 0" rpy="0 0 0" />
+            <material name="blue" />
+        </visual>
+        <collision>
+            <geometry>
+                <box size="0.005 0.03 0.03" />
             </geometry>
             <origin xyz="0.0 0.0 0.0" rpy="0.0 0.0 0.0" />
@@ -246,5 +246,5 @@
         <parent link="base_link" />
         <child link="camera" />
-        <origin xyz="0.14851 0.0022137 0.0975" />
+        <origin xyz="0.24851 0.0022137 0.0975" />
         <axis xyz="0 0 1" />
     </joint>
@@ -252,14 +252,12 @@
         <visual>
             <geometry>
-                <box size="0.01 0.1 0.02"/>
-            </geometry>
-            <origin xyz="0 0 0" rpy="0 0 0" />
-            <material name="black">
-                <color rgba="0.0 0.0 0.0 1.0" />
-            </material>
-        </visual>
-        <collision>
-            <geometry>
-                <box size="0.01 0.1 0.02"/>
+                <box size="0.01 0.1 0.02" />
+            </geometry>
+            <origin xyz="0 0 0" rpy="0 0 0" />
+            <material name="blue" />
+        </visual>
+        <collision>
+            <geometry>
+                <box size="0.01 0.1 0.02" />
             </geometry>
             <origin xyz="0.0 0.0 0.0" rpy="0.0 0.0 0.0" />
@@ -274,12 +272,12 @@
         <parent link="base_link" />
         <child link="real_sense" />
-        <origin xyz="0.19864 0.0038046 0.052021" />
-        <axis xyz="0 0 1" />
-    </joint>
-    <link name="realsense_depth"/>
+        <origin xyz="0.29864 0.0038046 0.052021" />
+        <axis xyz="0 0 1" />
+    </joint>
+    <link name="realsense_depth" />
     <joint name="realsense_depth_joint" type="fixed">
-            <origin xyz="0 0 0" rpy="-1.5708 0 -1.5708"/>
-            <parent link="real_sense"/>
-            <child link="realsense_depth"/>
+        <origin xyz="0 0 0" rpy="-1.5708 0 -1.5708" />
+        <parent link="real_sense" />
+        <child link="realsense_depth" />
     </joint>
     <link name="lidar">
@@ -289,7 +287,5 @@
             </geometry>
             <origin xyz="0 0 0" rpy="0 0 0" />
-            <material name="black">
-                <color rgba="0.0 0.0 0.0 1.0" />
-            </material>
+            <material name="blue" />
         </visual>
         <collision>
@@ -308,5 +304,5 @@
         <parent link="base_link" />
         <child link="lidar" />
-        <origin xyz="0.093603 0 0.12377" />
+        <origin xyz="0.193603 0 0.12377" />
         <axis xyz="0 0 1" />
     </joint>
@@ -314,14 +310,12 @@
         <visual>
             <geometry>
-                <box size="0.01 0.01 0.005"/>
-            </geometry>
-            <origin xyz="0 0 0" rpy="0 0 0" />
-            <material name="black">
-                <color rgba="0.0 0.0 0.0 1.0" />
-            </material>
-        </visual>
-        <collision>
-            <geometry>
-                <box size="0.01 0.01 0.005"/>
+                <box size="0.01 0.01 0.005" />
+            </geometry>
+            <origin xyz="0 0 0" rpy="0 0 0" />
+            <material name="blue" />
+        </visual>
+        <collision>
+            <geometry>
+                <box size="0.01 0.01 0.005" />
             </geometry>
             <origin xyz="0.0 0.0 0.0" rpy="0.0 0.0 0.0" />
@@ -339,4 +333,29 @@
         <axis xyz="0 0 1" />
     </joint>
-  <xacro:include filename="$(find racebot_description)/urdf/ackermann/ackermanncar.gazebo" />
+    <xacro:include filename="$(find racebot_description)/urdf/ackermann/ackermanncar.gazebo" />
+    <link name="grey_box">
+        <inertial>
+            <origin xyz="0 0 0" />
+            <mass value="0.5" />
+            <inertia ixx="6.64E-04" ixy="0" ixz="0" iyy="6.64E-04" iyz="0" izz="1.02E-03" />
+        </inertial>
+        <collision>
+            <origin rpy="0 0 0" xyz="0 0 0" />
+            <geometry>
+                <box size="0.4 0.5 0.05" />
+            </geometry>
+        </collision>
+        <visual>
+            <origin rpy="0 0 0" xyz="0 0 0" />
+            <geometry>
+                <box size="0.4 0.5 0.05" />
+            </geometry>
+            <material name="white" />
+        </visual>
+    </link>
+    <joint name="base_box" type="fixed">
+        <origin xyz="-0.2 0 0.05" rpy="0 0 0" />
+        <parent link="base_link" />
+        <child link="grey_box" />
+    </joint>
 </robot>

File: racebot_description/urdf/mecanum/mecanum_base.xacro (robot description, xacro)
@@ -59,4 +59,5 @@
             <axis xyz="0 1 0" />
             <limit effort="10" velocity="1000" />
+            <limit lower="-0.6" upper="0.6" effort="10" velocity="1000" />
         </joint>
         <link name="link_left_front">
@@ -92,5 +93,5 @@
             <origin xyz="0.40 -0.33 0" />
             <axis xyz="0 1 0" />
-            <limit effort="10" velocity="1000" />
+            <limit lower="-0.6" upper="0.6" effort="10" velocity="1000" />
         </joint>
         <link name="link_right_front">

Commit message: final

File: racebot_description/urdf/ackermann/ackermanncar.xacro (robot description, xacro)
@@ -304,5 +304,5 @@
         <parent link="base_link" />
         <child link="lidar" />
-        <origin xyz="0.193603 0 0.12377" />
+        <origin xyz="0.193603 0 0.32377" />
         <axis xyz="0 0 1" />
     </joint>

File: racebot_description/urdf/mecanum/mecanum_base.xacro (robot description, xacro)
@@ -210,5 +210,5 @@
             <parent link="base_link" />
             <child link="lidar" />
-            <origin xyz="0.193603 0 0.12377" />
+            <origin xyz="0.193603 0 0.32377" />
             <axis xyz="0 0 1" />
         </joint>
